File: hardware/T2101_rack_control.brd (EAGLE design)
At the start: 45.7 x 49.5 mm, 21 parts, among them Q1 IRFR220, Q2 600mA/40V, T1 DS18B20, U1 ATTINY84

Commit message: updat hdw
Parts:
- D1: value HSMR-C190 -> BLUE
- R1: value (none) -> 68
Connections:
- net N$2 renamed DPOS
Other:
- board text added: "+"
- board text added: "RST SCL MISO MOSI +5 GND"

Commit message: Fixes schematic issues
Parts:
- added C3: 4.7n, rcl:C0603K
- added D3: (no value), BeagleBone_Blue_R3:DIODE_SOD-123FL
- added R4, R5: 5k, rcl:R0603
- Q1: device transistor-fet:TO252 -> transistor-fet_220:TO252
- moved D2 10.9 mm to (10.2, 24.1)
- moved D1 8.89 mm to (30.5, 11.4)
Connections:
- net GND: now also C3.2, Q1.2; no longer Q1.3
- net MO: now also Q1.3; no longer Q1.2
- net RST: now also C3.1, D3.A, R5.2
- net TMP: now also R4.2
- net VCC5: now also D3.C, R4.1, R5.1
Routing:
- net DPOS: track 30.3 -> 3.23 mm
- net GND: track 54.7 -> 37.1 mm, vias 2 -> 4
- net VCC5: track 91.1 -> 106.2 mm, vias 3 -> 4
- net TMP: track 9.95 -> 20.7 mm
- net N$1: track 18.1 -> 7.55 mm
- net MISO: track 33.6 -> 43.7 mm, vias 0 -> 2
- net SCL: track 41.1 -> 31.2 mm, vias 2 -> 0
- net MO: track 30.2 -> 22.2 mm, vias 0 -> 1
- net RST: track 23.8 -> 27.6 mm
- net LED: track 18.1 -> 20.8 mm, vias 0 -> 2
- net MOSI: track 41.3 -> 40.7 mm
- net VCC12: track 34.7 -> 35.3 mm
- added copper zone on layer 1, net MO
- removed copper zone on layer 1, net GND
Other:
- board text added: "T2101"
- board text added: "v2"
