File: hardware/T2101_rack_control.sch (EAGLE design)
At the start: 21 parts, among them Q1 IRFR220, Q2 600mA/40V, T1 DS18B20, U1 ATTINY84

Commit message: updat hdw
Parts:
- D1: value HSMR-C190 -> BLUE
- R1: value (none) -> 68
Connections:
- net N$2 renamed DPOS
Changed lines of the file:
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@@
 <part name="P+1" library="supply1" library_urn="urn:adsk.eagle:library:371" deviceset="VCC" device="" value="VCC5"/>
 <part name="SUPPLY1" library="Fidget Spinner Example" library_urn="urn:adsk.eagle:library:9489508" deviceset="GND" device=""/>
-<part name="R1" library="rcl" library_urn="urn:adsk.eagle:library:334" deviceset="R-EU_" device="R0603" package3d_urn="urn:adsk.eagle:package:23555/3"/>
-<part name="D1" library="LED" library_urn="urn:adsk.eagle:library:12213040" deviceset="HSMR-C190" device="" package3d_urn="urn:adsk.eagle:package:10893503/2"/>
+<part name="R1" library="rcl" library_urn="urn:adsk.eagle:library:334" deviceset="R-EU_" device="R0603" package3d_urn="urn:adsk.eagle:package:23555/3" value="68"/>
+<part name="D1" library="LED" library_urn="urn:adsk.eagle:library:12213040" deviceset="HSMR-C190" device="" package3d_urn="urn:adsk.eagle:package:10893503/2" value="BLUE"/>
 <part name="SUPPLY2" library="Fidget Spinner Example" library_urn="urn:adsk.eagle:library:9489508" deviceset="GND" device=""/>
 <part name="Q1" library="transistor-fet" library_urn="urn:adsk.eagle:library:396" deviceset="SPD30P06P" device="TO252" package3d_urn="urn:adsk.eagle:package:28537/2" value="IRFR220"/>
@@
 </segment>
 </net>
-<net name="N$2" class="0">
+<net name="DPOS" class="0">
 <segment>
 <pinref part="R1" gate="G$1" pin="2"/>
@@
 <wire x1="78.74" y1="58.42" x2="83.82" y2="58.42" width="0.1524" layer="91"/>
 <junction x="78.74" y="53.34"/>
-<label x="83.82" y="58.42" size="1.778" layer="95" xref="yes"/>
+<label x="83.82" y="58.42" size="1.27" layer="95" xref="yes"/>
 </segment>
 <segment>
@@
 <wire x1="76.2" y1="50.8" x2="83.82" y2="50.8" width="0.1524" layer="91"/>
 <junction x="76.2" y="50.8"/>
-<label x="83.82" y="50.8" size="1.778" layer="95" xref="yes"/>
+<label x="83.82" y="50.8" size="1.27" layer="95" xref="yes"/>
 </segment>
 <segment>
 <pinref part="J6" gate="G$1" pin="3"/>
 <wire x1="17.78" y1="-2.54" x2="25.4" y2="-2.54" width="0.1524" layer="91"/>
-<label x="25.4" y="-2.54" size="1.778" layer="95" xref="yes"/>
+<label x="25.4" y="-2.54" size="1.27" layer="95" xref="yes"/>
 </segment>
 </net>
@@
 <pinref part="U1" gate="G$1" pin="(PCINT4/T1/SCL/USCK/ADC4)PA4"/>
 <wire x1="71.12" y1="48.26" x2="83.82" y2="48.26" width="0.1524" layer="91"/>
-<label x="83.82" y="48.26" size="1.778" layer="95" xref="yes"/>
+<label x="83.82" y="48.26" size="1.27" layer="95" xref="yes"/>
 </segment>
 <segment>
@@
 <pinref part="U1" gate="G$1" pin="(PCINT11/~RESET/DW)PB3"/>
 <wire x1="71.12" y1="68.58" x2="83.82" y2="68.58" width="0.1524" layer="91"/>
-<label x="83.82" y="68.58" size="1.778" layer="95" xref="yes"/>
-</segment>
-<segment>
+<label x="83.82" y="68.58" size="1.27" layer="95" xref="yes"/>
+</segment>
+<segment>

Commit message: Fixes schematic issues
Parts:
- added C3: 4.7n, rcl:C-EUC0603K
- added D3: (no value), BeagleBone_Blue_R3:DIODEDIODE-123FL
- added R4, R5: 5k, rcl:R-EU_R0603
- Q1: device transistor-fet:SPD30P06PTO252 -> transistor-fet_220:IFRU220NPBF
Connections:
- net GND: now also C3.2, Q1.S; no longer Q1.D
- net MO: now also Q1.D; no longer Q1.S
- net RST: now also C3.1, D3.A, R5.2
- net TMP: now also R4.2
- net VCC5: now also D3.C, R4.1, R5.1
Other:
- moved on the sheet: Q1
